File: Pix_Caster.sch (EAGLE design)
At the start: 198 parts, among them J1 2_POS_XH_DEV, J2 2_POS_XH_DEV, J3 13_POS_XH_DEV, J4 6_POS_XH_DEV, J5 8_POS_XH_DEV, Q1 2N2222, Q2 2n2222, U1 ESP_32_WROVER_I_PKG, U10 WDMX_NANO_DEV, U2 LD1117S33CTR_DEVLD1117S33CTR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

Commit message: first
Changed lines of the file:
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@@
 <part name="R33" library="Blizzard_Library" library_urn="urn:adsk.eagle:library:2665040" deviceset="0603_RES_DEV" device="3D" package3d_urn="urn:adsk.eagle:package:2685918/2" value="9K"/>
 <part name="VCC43" library="Blizzard_Library" library_urn="urn:adsk.eagle:library:2665040" deviceset="VCC" device="" value="3.3V"/>
+<part name="U$6" library="Blizzard_Library" library_urn="urn:adsk.eagle:library:2665040" deviceset="BLIZZARD_FRAME_DEV" device="">
+<attribute name="CDESC" value="Knob"/>
+</part>
+<part name="U$7" library="Blizzard_Library" library_urn="urn:adsk.eagle:library:2665040" deviceset="BLIZZARD_FRAME_DEV" device="">
+<attribute name="CDESC" value="Back Panel"/>
+</part>
+<part name="U$8" library="Blizzard_Library" library_urn="urn:adsk.eagle:library:2665040" deviceset="BLIZZARD_FRAME_DEV" device="">
+<attribute name="CDESC" value="LED Driver"/>
+</part>
 </parts>
 <sheets>
@@
 </instance>
 </instances>
+<busses>
+</busses>
+<nets>
+</nets>
+</sheet>
+<sheet>
+<plain>
+</plain>
+<instances>
+<instance part="U$6" gate="G$1" x="0" y="0" smashed="yes">
+<attribute name="CNAME" x="161.29" y="24.13" size="3.81" layer="94" font="vector"/>
+<attribute name="CDESC" x="161.29" y="17.78" size="3.81" layer="94" font="vector"/>
+<attribute name="LAST_DATE_TIME" x="161.29" y="11.43" size="3.81" layer="94" font="vector"/>
+<attribute name="SHEET" x="182.88" y="5.08" size="3.81" layer="94" font="vector"/>
+<attribute name="CDES" x="217.17" y="11.43" size="3.81" layer="94" font="vector"/>
+<attribute name="CREV" x="217.17" y="5.08" size="3.81" layer="94" font="vector"/>
+</instance>
+</instances>
+<busses>
+</busses>
+<nets>
+</nets>
+</sheet>
+<sheet>
+<plain>
+</plain>
+<instances>
+<instance part="U$7" gate="G$1" x="0" y="0" smashed="yes">
+<attribute name="CNAME" x="161.29" y="24.13" size="3.81" layer="94" font="vector"/>
+<attribute name="CDESC" x="161.29" y="17.78" size="3.81" layer="94" font="vector"/>
+<attribute name="LAST_DATE_TIME" x="161.29" y="11.43" size="3.81" layer="94" font="vector"/>
+<attribute name="SHEET" x="182.88" y="5.08" size="3.81" layer="94" font="vector"/>
+<attribute name="CDES" x="217.17" y="11.43" size="3.81" layer="94" font="vector"/>
+<attribute name="CREV" x="217.17" y="5.08" size="3.81" layer="94" font="vector"/>
+</instance>
+</instances>
+<busses>
+</busses>
+<nets>
+</nets>
+</sheet>
+<sheet>
+<plain>
+</plain>
+<instances>
+<instance part="U$8" gate="G$1" x="0" y="0" smashed="yes">
+<attribute name="CNAME" x="161.29" y="24.13" size="3.81" layer="94" font="vector"/>
+<attribute name="CDESC" x="161.29" y="17.78" size="3.81" layer="94" font="vector"/>
+<attribute name="LAST_DATE_TIME" x="161.29" y="11.43" size="3.81" layer="94" font="vector"/>
+<attribute name="SHEET" x="182.88" y="5.08" size="3.81" layer="94" font="vector"/>
+<attribute name="CDES" x="217.17" y="11.43" size="3.81" layer="94" font="vector"/>
+<attribute name="CREV" x="217.17" y="5.08" size="3.81" layer="94" font="vector"/>
+</instance>
+</instances>
